File: Hardware/CUBackplane.kicad_sch (KiCad schematic)
At the start: 49 parts, among them CON1 EXPANSION BUS, CON2 EXPANSION BUS, CON3 EXPANSION BUS, CON4 EXPANSION BUS, J1 +5V, J2 -12V, J3 +12V, J4 -5V, J5 +15V, J6 -15V, J7 GND

Commit message: Moved connector references
Parts:
- CON1, CON2, CON3, CON4: Mouser Link (none) -> https://mou.sr/4iZWKR4
